File: garbage-day-indicator.kicad_sch (KiCad schematic)
At the start: 18 parts, among them J1 Conn_01x16, J2 Conn_01x16

Commit message: Improve pcb layout
Parts:
- R1, R2, R3, R4, R5, R6, R7, R8, R9: footprint Resistor_SMD:R_0805_2012Metric -> Resistor_SMD:R_0603_1608Metric
- renumbered He1 to H2
Connections:
- net B1: now also J2.15 (Pin_15); no longer J2.7 (Pin_7)
- net B2: now also J2.10 (Pin_10); no longer J2.11 (Pin_11)
- net B3: now also J2.6 (Pin_6); no longer J1.9 (Pin_9)
- net G1: now also J1.9 (Pin_9); no longer J2.6 (Pin_6)
- net G2: now also J2.11 (Pin_11); no longer J2.10 (Pin_10)
- net G3: now also J2.7 (Pin_7); no longer J2.15 (Pin_15)
- net R2: now also J2.14 (Pin_14); no longer J2.9 (Pin_9)
- net R3: now also J2.9 (Pin_9); no longer J2.14 (Pin_14)
Changed lines of the file:
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@@
     (effects (font (size 1.27 1.27)) (justify right bottom))
   )
-  (label "B2" (at 119.38 95.25 0)
+  (label "G2" (at 119.38 95.25 0)
     (effects (font (size 1.27 1.27)) (justify left bottom))
   )
@@
     (effects (font (size 1.27 1.27)) (justify right bottom))
   )
-  (label "G3" (at 119.38 85.09 0)
+  (label "B1" (at 119.38 85.09 0)
     (effects (font (size 1.27 1.27)) (justify left bottom))
   )
@@
     (effects (font (size 1.27 1.27)) (justify right bottom))
   )
-  (label "G2" (at 119.38 97.79 0)
+  (label "B2" (at 119.38 97.79 0)
     (effects (font (size 1.27 1.27)) (justify left bottom))
   )
@@
     (effects (font (size 1.27 1.27)) (justify right bottom))
   )
-  (label "G1" (at 119.38 107.95 0)
-    (effects (font (size 1.27 1.27)) (justify left bottom))
-  )
-  (label "B1" (at 119.38 105.41 0)
+  (label "B3" (at 119.38 107.95 0)
+    (effects (font (size 1.27 1.27)) (justify left bottom))
+  )
+  (label "G3" (at 119.38 105.41 0)
     (effects (font (size 1.27 1.27)) (justify left bottom))
   )
@@
     (effects (font (size 1.27 1.27)) (justify right bottom))
   )
-  (label "B3" (at 104.14 100.33 0)
-    (effects (font (size 1.27 1.27)) (justify left bottom))
-  )
-  (label "R3" (at 119.38 87.63 0)
-    (effects (font (size 1.27 1.27)) (justify left bottom))
-  )
-  (label "R2" (at 119.38 100.33 0)
+  (label "G1" (at 104.14 100.33 0)
+    (effects (font (size 1.27 1.27)) (justify left bottom))
+  )
+  (label "R2" (at 119.38 87.63 0)
+    (effects (font (size 1.27 1.27)) (justify left bottom))
+  )
+  (label "R3" (at 119.38 100.33 0)
     (effects (font (size 1.27 1.27)) (justify left bottom))
   )
@@
     (property "Reference" "R9" (id 0) (at 194.31 107.95 90))
     (property "Value" "270" (id 1) (at 194.31 110.49 90))
-    (property "Footprint" "Resistor_SMD:R_0805_2012Metric" (id 2) (at 194.31 116.078 90)
+    (property "Footprint" "Resistor_SMD:R_0603_1608Metric" (id 2) (at 194.31 116.078 90)
       (effects (font (size 1.27 1.27)) hide)
     )
@@
   (symbol (lib_id "Mechanical:MountingHole_Pad") (at 73.66 99.06 0) (unit 1)
     (in_bom yes) (on_board yes) (fields_autoplaced)
-    (property "Reference" "He1" (id 0) (at 76.2 96.5199 0)
+    (property "Reference" "H2" (id 0) (at 76.2 96.5199 0)
       (effects (font (size 1.27 1.27)) (justify left))
     )
@@
     (property "Reference" "R6" (id 0) (at 162.56 107.95 90))
     (property "Value" "270" (id 1) (at 162.56 110.49 90))
-    (property "Footprint" "Resistor_SMD:R_0805_2012Metric" (id 2) (at 162.56 116.078 90)
+    (property "Footprint" "Resistor_SMD:R_0603_1608Metric" (id 2) (at 162.56 116.078 90)
       (effects (font (size 1.27 1.27)) hide)
     )
@@
     (property "Reference" "R7" (id 0) (at 194.31 85.09 90))
     (property "Value" "270" (id 1) (at 194.31 87.63 90))
-    (property "Footprint" "Resistor_SMD:R_0805_2012Metric" (id 2) (at 194.31 93.218 90)
+    (property "Footprint" "Resistor_SMD:R_0603_1608Metric" (id 2) (at 194.31 93.218 90)
       (effects (font (size 1.27 1.27)) hide)
     )
@@
     (property "Reference" "R1" (id 0) (at 134.62 85.09 90))
     (property "Value" "270" (id 1) (at 134.62 87.63 90))
-    (property "Footprint" "Resistor_SMD:R_0805_2012Metric" (id 2) (at 134.62 93.218 90)
+    (property "Footprint" "Resistor_SMD:R_0603_1608Metric" (id 2) (at 134.62 93.218 90)
       (effects (font (size 1.27 1.27)) hide)
     )
@@
     (property "Reference" "R5" (id 0) (at 162.56 96.52 90))
     (property "Value" "270" (id 1) (at 162.56 99.06 90))
-    (property "Footprint" "Resistor_SMD:R_0805_2012Metric" (id 2) (at 162.56 104.648 90)
+    (property "Footprint" "Resistor_SMD:R_0603_1608Metric" (id 2) (at 162.56 104.648 90)
       (effects (font (size 1.27 1.27)) hide)
     )
@@
     (property "Reference" "R8" (id 0) (at 194.31 96.52 90))
     (property "Value" "270" (id 1) (at 194.31 99.06 90))
-    (property "Footprint" "Resistor_SMD:R_0805_2012Metric" (id 2) (at 194.31 104.648 90)
+    (property "Footprint" "Resistor_SMD:R_0603_1608Metric" (id 2) (at 194.31 104.648 90)
       (effects (font (size 1.27 1.27)) hide)
     )
@@
     (property "Reference" "R2" (id 0) (at 134.62 96.52 90))
     (property "Value" "270" (id 1) (at 134.62 99.06 90))
-    (property "Footprint" "Resistor_SMD:R_0805_2012Metric" (id 2) (at 134.62 104.648 90)
+    (property "Footprint" "Resistor_SMD:R_0603_1608Metric" (id 2) (at 134.62 104.648 90)
       (effects (font (size 1.27 1.27)) hide)
     )
@@
     (property "Reference" "R3" (id 0) (at 134.62 107.95 90))
     (property "Value" "270" (id 1) (at 134.62 110.49 90))
-    (property "Footprint" "Resistor_SMD:R_0805_2012Metric" (id 2) (at 134.62 116.078 90)
+    (property "Footprint" "Resistor_SMD:R_0603_1608Metric" (id 2) (at 134.62 116.078 90)
       (effects (font (size 1.27 1.27)) hide)
     )
@@
     (property "Reference" "R4" (id 0) (at 162.56 85.09 90))
     (property "Value" "270" (id 1) (at 162.56 87.63 90))
-    (property "Footprint" "Resistor_SMD:R_0805_2012Metric" (id 2) (at 162.56 93.218 90)
+    (property "Footprint" "Resistor_SMD:R_0603_1608Metric" (id 2) (at 162.56 93.218 90)
       (effects (font (size 1.27 1.27)) hide)
     )
@@
       (reference "H1") (unit 1) (value "MountingHole_Pad") (footprint "MountingHole:MountingHole_3.2mm_M3_DIN965_Pad")
     )
+    (path "/247c1f31-f3c3-4b0c-881d-e6da3f354c06"
+      (reference "H2") (unit 1) (value "MountingHole_Pad") (footprint "MountingHole:MountingHole_3.2mm_M3_DIN965_Pad")
+    )
     (path "/d78efa19-a943-4403-8264-7bb3f9955ed3"
       (reference "H3") (unit 1) (value "MountingHole_Pad") (footprint "MountingHole:MountingHole_3.2mm_M3_DIN965_Pad")
@@
       (reference "H4") (unit 1) (value "MountingHole_Pad") (footprint "MountingHole:MountingHole_3.2mm_M3_DIN965_Pad")
     )
-    (path "/247c1f31-f3c3-4b0c-881d-e6da3f354c06"
-      (reference "He1") (unit 1) (value "MountingHole_Pad") (footprint "MountingHole:MountingHole_3.2mm_M3_DIN965_Pad")
-    )
     (path "/6d8c8373-0d56-457e-8bc2-aa34a7d9f788"
       (reference "J1") (unit 1) (value "Conn_01x16") (footprint "Connector_PinSocket_2.54mm:PinSocket_1x16_P2.54mm_Vertical")
@@
     )
     (path "/84347e16-4e8f-4fcc-85b9-978fe05b8e8a"
-      (reference "R1") (unit 1) (value "270") (footprint "Resistor_SMD:R_0805_2012Metric")
+      (reference "R1") (unit 1) (value "270") (footprint "Resistor_SMD:R_0603_1608Metric")
     )
     (path "/de36f986-78ec-4473-92fb-dc5b172215a3"
-      (reference "R2") (unit 1) (value "270") (footprint "Resistor_SMD:R_0805_2012Metric")
+      (reference "R2") (unit 1) (value "270") (footprint "Resistor_SMD:R_0603_1608Metric")
     )
     (path "/e336fc40-d21e-4eff-a20e-68ee022dc7b4"
-      (reference "R3") (unit 1) (value "270") (footprint "Resistor_SMD:R_0805_2012Metric")
+      (reference "R3") (unit 1) (value "270") (footprint "Resistor_SMD:R_0603_1608Metric")
     )
     (path "/f209c549-12ec-47c8-af85-a977e2854a32"
-      (reference "R4") (unit 1) (value "270") (footprint "Resistor_SMD:R_0805_2012Metric")
+      (reference "R4") (unit 1) (value "270") (footprint "Resistor_SMD:R_0603_1608Metric")
     )
     (path "/aa899e20-9875-4f0d-8b73-3530e83b67c6"
-      (reference "R5") (unit 1) (value "270") (footprint "Resistor_SMD:R_0805_2012Metric")
+      (reference "R5") (unit 1) (value "270") (footprint "Resistor_SMD:R_0603_1608Metric")
     )
     (path "/3361e817-06fc-40f1-a34b-db1cd038700f"
-      (reference "R6") (unit 1) (value "270") (footprint "Resistor_SMD:R_0805_2012Metric")
+      (reference "R6") (unit 1) (value "270") (footprint "Resistor_SMD:R_0603_1608Metric")
     )
     (path "/6fd4149c-8bf9-4fcd-b6c3-5497aa46a3ca"
-      (reference "R7") (unit 1) (value "270") (footprint "Resistor_SMD:R_0805_2012Metric")
+      (reference "R7") (unit 1) (value "270") (footprint "Resistor_SMD:R_0603_1608Metric")
     )
     (path "/d9b77527-abd6-4473-a0e5-c4d5a5abbf94"
-      (reference "R8") (unit 1) (value "270") (footprint "Resistor_SMD:R_0805_2012Metric")
+      (reference "R8") (unit 1) (value "270") (footprint "Resistor_SMD:R_0603_1608Metric")
     )
     (path "/02517c45-467b-4134-bb7e-696380a57130"
-      (reference "R9") (unit 1) (value "270") (footprint "Resistor_SMD:R_0805_2012Metric")
-    )
-  )
+      (reference "R9") (unit 1) (value "270") (footprint "Resistor_SMD:R_0603_1608Metric")
+    )
+  )
